File: hardware/pcb/kiwiigo.kicad_pcb (KiCad board)
At the start: 2 copper layers, 100 x 50 mm, 27 parts, among them J1 Conn_01x02, Q1 IRLML6402, U1 NEO-M8N, U2 RFM95W-915S2, U3 MCP73831-2-OT, U4 AP2112K-3.3, U5 DS3231SN#_C722469

Commit message: gitignore
gittyignoe
Parts:
- U1: footprint RF_GPS:ublox_NEO -> easyeda2kicad:GPSM-SMD_NEO-M8N
- turned U1 to -90 degrees
Routing:
- net /GPS_TX: track 100.7 -> 101.4 mm
