File: hardware/pcb/kiwiigo.kicad_sch (KiCad schematic)
At the start: 19 parts, among them J1 Conn_01x02, Q1 IRLML6402, U1 NEO-M8N, U2 RFM95W-915S2, U3 MCP73831-2-OT, U4 AP2112K-3.3, U5 DS3231SN#_C722469

Commit message: gitignore
gittyignoe
Parts:
- U1: footprint RF_GPS:ublox_NEO -> easyeda2kicad:GPSM-SMD_NEO-M8N
Connections:
- net +3.3V: no longer A1.36 (3V3)
- net DIN renamed RGB_GLOW
- no-connect marks 1 -> 42
Other:
- note removed: "transmit & receive"
- moved on the sheet: J1, Q1, R1, R2, R3, U2, U3, U4, U5
